Commit message: up

File: launch/mowbot_robot_launch/urdf/mowbot.xacro (robot description, xacro)
@@ -1,9 +1,9 @@
 <?xml version="1.0"?>
-<robot name="vehicle" xmlns:xacro="http://ros.org/wiki/xacro">
-  <xacro:arg name="mowbot_model" default=""/>
+<robot name="robot" xmlns:xacro="http://ros.org/wiki/xacro">
+  <xacro:arg name="robot_model" default=""/>
   <xacro:arg name="sensor_model" default=""/>
-  <!-- vehicle -->
-  <xacro:property name="mowbot_model_property" value="$(arg vehicle_model)"/>
-  <xacro:include filename="$(find ${mowbot_model_property}_description)/urdf/mowbot.xacro"/>
+  <!-- robot -->
+  <xacro:property name="robot_model_property" value="$(arg robot_model)"/>
+  <xacro:include filename="$(find ${robot_model_property}_description)/urdf/robot.xacro"/>
   <!-- sensors -->
   <xacro:property name="sensor_model_property" value="$(arg sensor_model)"/>
