Commit message: gazebo robot description

File: launch/mowbot_robot_launch/urdf/robot.xacro (robot description, xacro)
@@ -7,5 +7,5 @@
   <xacro:include filename="$(find ${robot_model_property}_description)/urdf/robot.xacro"/>
   <!-- sensors -->
-  <xacro:property name="sensor_model_property" value="$(arg sensor_model)"/>
-  <xacro:include filename="$(find ${sensor_model_property}_description)/urdf/sensors.xacro"/>
+  <!-- <xacro:property name="sensor_model_property" value="$(arg sensor_model)"/>
+  <xacro:include filename="$(find ${sensor_model_property}_description)/urdf/sensors.xacro"/> -->
 </robot>

Commit message: up

File: launch/mowbot_robot_launch/urdf/robot.xacro (robot description, xacro)
@@ -7,5 +7,5 @@
   <xacro:include filename="$(find ${robot_model_property}_description)/urdf/robot.xacro"/>
   <!-- sensors -->
-  <!-- <xacro:property name="sensor_model_property" value="$(arg sensor_model)"/>
-  <xacro:include filename="$(find ${sensor_model_property}_description)/urdf/sensors.xacro"/> -->
+  <xacro:property name="sensor_model_property" value="$(arg sensor_model)"/>
+  <xacro:include filename="$(find ${sensor_model_property}_description)/urdf/sensors.xacro"/>
 </robot>
